Commit message: Calibrate phone tilt from gravity: rpy=(90,-10.7,90) not (0,-60,90)

File: ros2_ws/src/tank_description/urdf/tank.urdf (robot description, URDF)
Before this commit: robot rovac_tank, 12 links, 11 joints
Joints:
- joint phone_imu_joint: origin xyz=-0.08 0.0 0.234 rpy=0 -1.0472 1.5708 -> xyz=-0.08 0.0 0.234 rpy=1.5708 -0.1868 1.5708
