Commit message: Add EKF sensor fusion, updated URDF with measured dimensions, robot calibration doc
EKF Fusion (config/ekf_params.yaml + scripts/ekf_launch.py):
- Fuses wheel odometry (/odom) with phone IMU (/phone/imu/relay)
- Output: /odometry/filtered — improved localization with gyro correction
- 2D mode, imu0_relative=true to avoid yaw fighting
- Launch: ./mac_brain_launch.sh ekf

URDF updates (tank.urdf):
- LIDAR: corrected to xyz=(0.08, 0, 0.11) from ruler measurement (was 0.125)
- Added phone_imu_link at (-0.07, 0, 0.21) with rpy=(0, 1.047, 1.571)
  60deg forward tilt + 90deg landscape rotation
- Added phone_gps_link and phone_camera_link as children of phone_imu
- Removed old camera_link and stereo_camera (replaced by phone)

Robot dimensions document (docs/robot_dimensions.md):
- Complete measured dimensions from ruler/level photos
- G1 Tank chassis specs, LIDAR position, phone mount geometry
- Phone IMU axis mapping (Android portrait → ROS REP-103)
- TF tree diagram, calibration notes

Co-Authored-By: Claude Opus 4.6 (1M context) <noreply@anthropic.com>

File: ros2_ws/src/tank_description/urdf/tank.urdf (robot description, URDF)
Before this commit: robot rovac_tank, 11 links, 10 joints
Links:
- removed link camera_link
- removed link stereo_camera
- added link phone_camera_link
- added link phone_gps_link
- added link phone_imu_link; visual box size=0.164 0.078 0.008
Joints:
- removed joint camera_joint
- removed joint stereo_camera_joint
- added joint phone_camera_joint: type fixed, parent phone_imu_link, child phone_camera_link, origin xyz=0 0.07 -0.004 rpy=0 0 0
- added joint phone_gps_joint: type fixed, parent phone_imu_link, child phone_gps_link, origin xyz=0 0.04 0 rpy=0 0 0
- added joint phone_imu_joint: type fixed, parent base_link, child phone_imu_link, origin xyz=-0.07 0.0 0.21 rpy=0 1.0472 1.5708
- joint laser_joint: origin xyz=0 0 0.125 rpy=0 0 0 -> xyz=0.08 0 0.11 rpy=0 0 0

Commit message: Fix phone tilt direction: screen faces REAR, camera faces FORWARD
CRITICAL CORRECTION: Phone pitch was +60deg (forward), should be -60deg (backward).
- Phone screen faces the REAR of the robot
- Phone rear camera faces FORWARD (driving direction)
- Zenith angle 330deg = tilted 60deg from vertical toward the rear
- URDF pitch: -1.0472 rad (was +1.0472)

Updated all documents: URDF, wireframe diagram, dimensions doc.

Co-Authored-By: Claude Opus 4.6 (1M context) <noreply@anthropic.com>

File: ros2_ws/src/tank_description/urdf/tank.urdf (robot description, URDF)
Before this commit: robot rovac_tank, 12 links, 11 joints
Joints:
- joint phone_imu_joint: origin xyz=-0.07 0.0 0.21 rpy=0 1.0472 1.5708 -> xyz=-0.07 0.0 0.21 rpy=0 -1.0472 1.5708

Commit message: Correct all robot dimensions from physical measurements
Major corrections based on user's detailed measurements:
- base_link height: 20mm from ground (motor shaft), was 50mm
- base_footprint offset: -0.02m, was -0.05m
- LIDAR X: +0.015m (nearly centered, 95mm from front edge), was +0.08m
- LIDAR Z: +0.1325m (scan plane at 152.5mm from ground), was +0.11m
- Phone Z: +0.234m (center at 254mm from ground), was +0.21m
- Phone X: -0.08m, was -0.07m
- Robot width: 245mm (outer tracks), was 170mm
- Robot length: ~220mm, was 230mm
- Chassis box visual updated to 220x245mm

Added platform details:
- Lower platform at 40mm (ESP32 + battery)
- Upper platform tapered: 140mm front, 100mm rear
- Max robot height: 295mm (phone top)

Co-Authored-By: Claude Opus 4.6 (1M context) <noreply@anthropic.com>

File: ros2_ws/src/tank_description/urdf/tank.urdf (robot description, URDF)
Before this commit: robot rovac_tank, 12 links, 11 joints
Links:
- link base_link: geometry visual box size=0.22 0.245 0.10
Joints:
- joint base_footprint_joint: origin xyz=0 0 -0.05 rpy=0 0 0 -> xyz=0 0 -0.02 rpy=0 0 0
- joint laser_joint: origin xyz=0.08 0 0.11 rpy=0 0 0 -> xyz=0.015 0 0.1325 rpy=0 0 0
- joint phone_imu_joint: origin xyz=-0.07 0.0 0.21 rpy=0 -1.0472 1.5708 -> xyz=-0.08 0.0 0.234 rpy=0 -1.0472 1.5708

Commit message: Fix EKF prerequisites: odom relay, frame_id matching, QoS bridging
- Add /odom relay (best_effort → reliable /odom/reliable) to tf_relay.py
  for robot_localization EKF compatibility
- EKF config: use /odom/reliable and /phone/imu (not relay)
- URDF: rename frames to match phone app (phone_imu, phone_gps, phone_camera)
  without _link suffix — matches frame_id in published messages

Co-Authored-By: Claude Opus 4.6 (1M context) <noreply@anthropic.com>

File: ros2_ws/src/tank_description/urdf/tank.urdf (robot description, URDF)
Before this commit: robot rovac_tank, 12 links, 11 joints
Links:
- removed link phone_camera_link
- removed link phone_gps_link
- removed link phone_imu_link
- added link phone_camera
- added link phone_gps
- added link phone_imu; visual box size=0.164 0.078 0.008
Joints:
- joint phone_camera_joint: child phone_camera_link -> phone_camera; parent phone_imu_link -> phone_imu
- joint phone_gps_joint: child phone_gps_link -> phone_gps; parent phone_imu_link -> phone_imu
- joint phone_imu_joint: child phone_imu_link -> phone_imu

Commit message: Integrate BNO055 IMU into motor controller with EKF fusion
Full end-to-end integration of Adafruit BNO055 9-axis IMU:

Firmware (ESP32 motor controller):
- BNO055 driver (bno055.c/h) using new ESP-IDF I2C master driver
  with scl_wait_us=5000 for clock-stretching compatibility
- Migrated OLED driver to new I2C master API (thread-safe, no mutex)
- /imu/data publisher (sensor_msgs/Imu, 20Hz, best_effort)
- Calibration status in /diagnostics KV pairs
- Calibration persistence via NVS (22-byte profile auto-saved at 3/3/3/3)
- Gyro-assisted heading correction in PID loop (KP=0.5)
- Interrupt-driven reads (GPIO25) with 50Hz polling fallback
- MAX_PUBLISHERS increased to 4 in app-colcon.meta

ROS2 pipeline:
- imu_relay.py: /imu/data → /imu/data_reliable (separate topic)
- odom_relay.py: /odom → /odom_reliable (FIXED: separate topic
  prevents double-delivery that caused 40° EKF yaw oscillation)
- EKF config: fuses /odom_reliable + /imu/data_reliable
  (yaw differential + vyaw from gyro)
- URDF: imu_link with face-down mounting (rpy=π,0,0)
- Systemd: rovac-edge-imu-relay.service, updated ekf.service deps

Monitoring:
- Command center TUI: BNO055 panel in sensors, dashboard indicator
- Process manager: added relay services to PI_SERVICES list

Also includes: BNO055 test firmware (hardware/bno055_test/),
RPLIDAR C1 docs, robot annotated images, map files.

Co-Authored-By: Claude Opus 4.6 (1M context) <noreply@anthropic.com>

File: ros2_ws/src/tank_description/urdf/tank.urdf (robot description, URDF)
Before this commit: robot rovac_tank, 12 links, 11 joints
Links:
- added link front_indicator; visual box size=0.06 0.04 0.02
- link laser_frame: geometry visual box size=0.0556 0.0556 0.0413
Joints:
- added joint front_indicator_joint: type fixed, parent base_link, child front_indicator, origin xyz=0.13 0 0.04 rpy=0 0 0
- joint imu_joint: origin xyz=0 0 0.02 rpy=0 0 0 -> xyz=0 0 0.02 rpy=3.14159 0 0
- joint laser_joint: origin xyz=0.015 0 0.1325 rpy=0 0 0 -> xyz=0.015 0 0.12 rpy=0 0 0

Commit message: Coverage: pad-aware planner + ground-truth tracker + URDF link
Core change: shift the autonomous-vacuum problem from "robot covers
floor" to "vacuum pad covers floor". The pad is only 10.5 cm wide and
sits 18.8 cm forward of base_link, so the previous 30 cm row spacing
was leaving ~20 cm un-vacuumed strips between rows.

URDF
----
Add vacuum_pad_link (5.4×10.5 cm box) parented to base_footprint at
+0.1878 m forward, +0.0025 m up. Dimensions and offset measured from
ruler photos and CLAUDE.md geometry. Parented to base_footprint (not
base_link) so the cells-on-floor math is purely 2D.

coverage_node.py
----------------
Replace robot-width assumptions with pad geometry:
  pad_width             = 0.10478 m  (new param)
  pad_overlap_fraction  = 0.33       (new param, conservative default)
  swath_width           = pad_width × (1 - overlap)  = 7.0 cm by default
  robot_radius          = 0.13 m (down from 0.17 — body half-width only;
                                  pad sticks forward into inflation zone
                                  on purpose so it can reach near walls)
  min_span_length       = 0.20 m (was 0.25)
  goal_tolerance        = 0.20 m (was 0.25 — tighter so rows stay on-line)

coverage_tracker.py (new)
-------------------------
Independent verifier. Subscribes to /map + TF, projects the pad rectangle
onto the map grid every 100 ms, marks visited cells, publishes:
  /coverage/visited     (OccupancyGrid, transient_local) — visited cells
  /coverage/pad_polygon (PolygonStamped)                  — live pad outline
Publishes a coverage % every cycle.

Foxglove layout
---------------
Render /coverage/visited as a green overlay on the SLAM map and
/coverage/pad_polygon as a magenta outline. Add TRACKER indicator panel.

Run sequence (full instructions follow in chat).

Co-Authored-By: Claude Opus 4.7 (1M context) <noreply@anthropic.com>

File: ros2_ws/src/tank_description/urdf/tank.urdf (robot description, URDF)
Before this commit: robot rovac_tank, 13 links, 12 joints
Links:
- added link vacuum_pad_link; visual box size=0.05398 0.10478 0.005
Joints:
- added joint vacuum_pad_joint: type fixed, parent base_footprint, child vacuum_pad_link, origin xyz=0.1878 0 0.0025 rpy=0 0 0

Commit message: Foxglove + diagnostics polish: stable indicators, clean 3D, fix lifecycle list
Four issues from the live preview, fixed together so the next launch
is clean for live driving:

1) URDF cleanup — retired hardware removed
   Strip phone_imu / phone_camera / phone_gps and the entire
   super_sensor_link tree (4 ultrasonic visualization links). These
   were retired weeks ago (BNO055 replaces phone IMU; ESP32 sensor hub
   replaces super_sensor) but still rendered as TF labels overlaid on
   the robot in the 3D panel. URDF now has 6 links instead of 14.

2) Stable per-source diagnostic indicators (the flickering MOTOR fix)
   /diagnostics is one topic shared by N publishers. A Foxglove indicator
   reading /diagnostics.status[0].level flickers because status[0] is
   whichever source spoke last — motor (level 0), sensor hub (level 1),
   ekf, lifecycle_manager etc. all rotate through that slot.

   New: scripts/diagnostics_splitter.py subscribes /diagnostics, filters
   each DiagnosticStatus by .name, and republishes on dedicated latched
   topics:
     /diag/motor          ← "ROVAC Motor Serial"
     /diag/sensor_hub     ← "ROVAC Sensor Hub"
     /diag/ekf            ← ekf_node
     /diag/nav2_lifecycle ← lifecycle_manager_navigation
   These are TRANSIENT_LOCAL so a Foxglove panel that connects later
   still sees the latest known status.

   Layout changed: MOTOR indicator now reads /diag/motor.level (stable).
   Added a SENSOR HUB indicator alongside.

   Runs on Pi as rovac-edge-diagnostics-splitter.service; added to
   install_pi_systemd.sh. Pi services on /diagnostics speak first; the
   splitter routes them; Mac-side ekf/nav2 diagnostics get routed too
   when those run.

3) /smoother_server doesn't exist — fix lifecycle node list
   Nav2 has two distinct smoothers: nav2_smoother (smoother_server) and
   nav2_velocity_smoother (velocity_smoother). nav2_launch.py only uses
   the latter. Both nav2_recover.py and verify_and_recover_nav2 had
   /smoother_server in the check list, so verification always saw one
   "blank" node. Updated both to the correct 8-node list from
   nav2_launch.py: map_server, amcl, controller_server, planner_server,
   behavior_server, velocity_smoother, waypoint_follower, bt_navigator.

4) Hide TF labels in 3D view
   Set scene.labelScaleFactor=0 and transforms.axisScale=0.0 in the
   layout. With showLabel:false alone, individual frames could still
   override; setting label scale to 0 globally collapses them all.

Co-Authored-By: Claude Opus 4.7 (1M context) <noreply@anthropic.com>

File: ros2_ws/src/tank_description/urdf/tank.urdf (robot description, URDF)
Before this commit: robot rovac_tank, 14 links, 13 joints
Links:
- removed link phone_camera
- removed link phone_gps
- removed link phone_imu
- removed link super_sensor_link
- removed link super_sensor_link/front_bottom_link
- removed link super_sensor_link/front_top_link
- removed link super_sensor_link/left_link
- removed link super_sensor_link/right_link
Joints:
- removed joint phone_camera_joint
- removed joint phone_gps_joint
- removed joint phone_imu_joint
- removed joint super_sensor_joint
- removed joint us_front_bottom_joint
- removed joint us_front_top_joint
- removed joint us_left_joint
- removed joint us_right_joint

Commit message: hardware: stereo cameras — dual Pi 5 CSI OV5647 NoIR replaces USB webcam stack
Retire the legacy USB-webcam stereo system (cv2.VideoCapture + Python
StereoSGBM + obstacle detector) and replace with an industry-standard ROS2
stereo bringup using libcamera + camera_ros for two Raspberry Pi NoIR
Camera Module v1 (OV5647) sensors on the Pi 5's native CSI ports.

New ROS2 package: rovac_stereo_camera (launch + placeholder camera_info).
New systemd service: rovac-edge-stereo-cameras (wired into rovac-edge.target).
New URDF frames: stereo_camera_link, stereo_{left,right}_camera_{link,
optical_frame} — REP-103 compliant, placeholder geometry pending mount.
New reproducibility script: scripts/build_pi_libcamera.sh — idempotent
build of Pi-patched libcamera 0.5.2 + camera_ros 0.6.0, plus a 'libcamera'
subcommand in install_pi_systemd.sh and a camera_ros pin in external.repos.

Topics published: /stereo/{left,right}/{image_raw, image_raw/compressed,
camera_info} — matches stereo_image_proc consumer expectations so Phase 3
disparity/pointcloud composition is a one-line uncomment away (see
commented blocks in stereo_cameras.launch.py).

Architecture notes:
- Pi-patched libcamera 0.5.2 built from source to /opt/rpi-libcamera.
  Ubuntu's 0.2.0 lacks Pi 5 pisp pipeline support; OSRF's 0.7.0 ABI
  doesn't match the Pi-tree kernel CFE driver. The Pi-stable 0.5.2 fork
  is paired with the matching kernel CFE driver.
- camera_ros 0.6.0 built from source (apt binary links against the wrong
  libcamera SONAME 0.7).
- Two ComposableNodeContainers (one per camera) — libcamera's
  CameraManager is a per-process singleton.
- /boot/firmware/config.txt updated with explicit dtoverlay=ov5647,cam0
  + cam1 (camera_auto_detect=1 fails on dual-CSI Pi 5 + Ubuntu Noble).

Retired files moved to archive/legacy_hardware/stereo_cameras_usb/.
Removed systemd units: rovac-edge-stereo-depth, rovac-edge-stereo-obstacle,
rovac-edge-stereo.target, rovac-edge-webcam.

Co-Authored-By: Claude Opus 4.7 (1M context) <noreply@anthropic.com>

File: ros2_ws/src/tank_description/urdf/tank.urdf (robot description, URDF)
Before this commit: robot rovac_tank, 6 links, 5 joints
Links:
- added link stereo_camera_link
- added link stereo_left_camera_link; visual box size=0.025 0.024 0.009
- added link stereo_left_camera_optical_frame
- added link stereo_right_camera_link; visual box size=0.025 0.024 0.009
- added link stereo_right_camera_optical_frame
Joints:
- added joint stereo_camera_joint: type fixed, parent base_link, child stereo_camera_link, origin xyz=0.10 0 0.10 rpy=0 0 0
- added joint stereo_left_camera_joint: type fixed, parent stereo_camera_link, child stereo_left_camera_link, origin xyz=0 0.030 0 rpy=0 0 0
- added joint stereo_left_camera_optical_joint: type fixed, parent stereo_left_camera_link, child stereo_left_camera_optical_frame, origin xyz=0 0 0 rpy=-1.5707963 0 -1.5707963
- added joint stereo_right_camera_joint: type fixed, parent stereo_camera_link, child stereo_right_camera_link, origin xyz=0 -0.030 0 rpy=0 0 0
- added joint stereo_right_camera_optical_joint: type fixed, parent stereo_right_camera_link, child stereo_right_camera_optical_frame, origin xyz=0 0 0 rpy=-1.5707963 0 -1.5707963

Commit message: fix: complete front/rear URDF rework — rotate laser_joint to match
The 2026-05-18 rework redefining the robot's front (red-box end = +X,
LIDAR/RPi/camera stack = rear/-X) was deployed but never committed. It
also missed one thing: it moved the RPLIDAR joint position from +X to
-X but left rpy at "0 0 0". The physical RPLIDAR C1's 0° azimuth points
toward the lidar-stack end — now the rear — so /scan rendered 180°
rotated vs the model in Foxglove and RViz2 (a person behind the robot
appeared in front of it).

This commit lands the full rework plus the fix:
- laser_joint rpy="0 0 3.14159" — aligns /scan with base_link
- vacuum_pad_link removed; rpi_link + rpi_battery_link added
- LIDAR / stereo stack repositioned to the rear deck (-X)
- corrected a stale comment claiming a nonexistent odom_rotate_180 param

Verified: live TF base_link->laser_frame yaw = 180°; rear-approach scan
test registers correctly. Firmware and /odom were already correct.

Co-Authored-By: Claude Opus 4.7 (1M context) <noreply@anthropic.com>

File: ros2_ws/src/tank_description/urdf/tank.urdf (robot description, URDF)
Before this commit: robot rovac_tank, 11 links, 10 joints
Links:
- removed link vacuum_pad_link
- added link rpi_battery_link; visual box size=0.090 0.070 0.025
- added link rpi_link; visual box size=0.085 0.056 0.020
Joints:
- removed joint vacuum_pad_joint
- added joint rpi_battery_joint: type fixed, parent base_link, child rpi_battery_link, origin xyz=-0.065 0 0.0625 rpy=0 0 0
- added joint rpi_joint: type fixed, parent base_link, child rpi_link, origin xyz=-0.065 0 0.085 rpy=0 0 0
- joint laser_joint: origin xyz=0.015 0 0.12 rpy=0 0 0 -> xyz=-0.065 0 0.118 rpy=0 0 3.14159
- joint stereo_camera_joint: origin xyz=0.10 0 0.10 rpy=0 0 0 -> xyz=-0.065 0 0.150 rpy=0 0 0

Commit message: feat: add sensor-hub TF frames to URDF; obstacle node reads poses from TF
URDF (tank.urdf):
- add 6 sensor frames — us_front/rear/left/right_link + cliff_front/
  cliff_rear_link — positioned and aimed from 2026-05-18 measurements.
  sensor_msgs/Range projects along each frame's +X, so joint rpy fans
  the ultrasonic cones outward and pitches the cliff cones at the floor.
- update robot dimensions (241.3 x 240 mm), IMU (+95.25mm X), rear-stack
  X (-76.2mm), and stereo-camera height (355.6mm above the floor).

obstacle_avoidance_node.py:
- read the 4 ultrasonic poses (position + facing direction) live from
  TF (base_link -> us_*_link) instead of hardcoding them; the URDF is
  now the single source of truth. Removes a stale hardcoded front
  position (0.250 m — geometrically impossible for a 241mm robot).
- min_valid stays hardcoded (tuning, not geometry); commented that the
  front value needs re-tuning for the new 76mm mount height.

Verified on the robot: all 8 frames live in TF; the obstacle node logs
"All ultrasonic frames resolved from TF".

Co-Authored-By: Claude Opus 4.7 (1M context) <noreply@anthropic.com>

File: ros2_ws/src/tank_description/urdf/tank.urdf (robot description, URDF)
Before this commit: robot rovac_tank, 12 links, 11 joints
Links:
- added link cliff_front_link; visual box size=0.020 0.011 0.007
- added link cliff_rear_link; visual box size=0.020 0.011 0.007
- added link us_front_link; visual box size=0.020 0.045 0.015
- added link us_left_link; visual box size=0.020 0.045 0.015
- added link us_rear_link; visual box size=0.020 0.045 0.015
- added link us_right_link; visual box size=0.020 0.045 0.015
- link base_link: geometry visual box size=0.2413 0.240 0.10
Joints:
- added joint cliff_front_joint: type fixed, parent base_link, child cliff_front_link, origin xyz=0.12065 0 0.0308 rpy=0 1.5707963 0
- added joint cliff_rear_joint: type fixed, parent base_link, child cliff_rear_link, origin xyz=-0.12065 0 0.0308 rpy=0 1.5707963 0
- added joint us_front_joint: type fixed, parent base_link, child us_front_link, origin xyz=0.12065 0 0.0562 rpy=0 0 0
- added joint us_left_joint: type fixed, parent base_link, child us_left_link, origin xyz=0 0.070 0.0562 rpy=0 0 1.5707963
- added joint us_rear_joint: type fixed, parent base_link, child us_rear_link, origin xyz=-0.12065 0 0.195 rpy=0 0 3.14159
- added joint us_right_joint: type fixed, parent base_link, child us_right_link, origin xyz=0 -0.070 0.0562 rpy=0 0 -1.5707963
- joint imu_joint: origin xyz=0 0 0.02 rpy=3.14159 0 0 -> xyz=0.09525 0 0.02 rpy=3.14159 0 0
- joint laser_joint: origin xyz=-0.065 0 0.118 rpy=0 0 3.14159 -> xyz=-0.0762 0 0.118 rpy=0 0 3.14159
- joint rpi_battery_joint: origin xyz=-0.065 0 0.0625 rpy=0 0 0 -> xyz=-0.0762 0 0.0625 rpy=0 0 0
- joint rpi_joint: origin xyz=-0.065 0 0.085 rpy=0 0 0 -> xyz=-0.0762 0 0.085 rpy=0 0 0
- joint stereo_camera_joint: origin xyz=-0.065 0 0.150 rpy=0 0 0 -> xyz=-0.0762 0 0.3356 rpy=0 0 0
